File: Sapflow/smart_probe/smart_probe.sch (EAGLE design)
At the start: 33 parts, among them IC1 MCP3424-E_SL, IC2 PCA9615DPJ

Commit message: Removed duplicate versions
Parts:
- removed IC2: PCA9615DPJ, PCA9615DPJ:PCA9615DPJ
- removed R12, R13: 0, rcl:R-US_R0603
- removed R18, R19, R21: 600, rcl:R-US_R0603
- removed R20: 120, rcl:R-US_R0603
- removed SV1: (no value), con-lstb:MA04-2
- removed SV3: (no value), con-lstb:MA05-2
- added INPUT: (no value), better_header:MA03-2
- added LED1, LED2: (no value), led:LEDCHIP-LED0805
- added PROBE: (no value), better_header:MA04-2
- added SJ1, SJ2, SJ3, SJ4: (no value), jumper:SJ
- added SPARKFUN: (no value), SparkX:I2C_STANDARD_NO_SILK
- C1, C2, C3, C4, C5, C6, C7, C8: device rcl:C-USC0603 -> rcl:C-USC0805
- R1, R10, R11, R14, R15, R2, R3, R4, R5, R6, R7, R8, R9: device rcl:R-US_R0603 -> rcl:R-US_R0805
- R16: value 600 -> 5k; device rcl:R-US_R0603 -> rcl:R-US_R0805
- R17: value 120 -> 1.5k; device rcl:R-US_R0603 -> rcl:R-US_R0805
Connections:
- removed net ADR0: IC1.ADR0, R13.1
- removed net ADR1: IC1.ADR1, R12.1
- removed net AGND: R7.2
- removed net AVDD: C6.1, C7.1, R10.1, R11.1, R12.1, R8.2
- removed net CLK+: IC2.DSCLM, R19.1, R20.2, SV3.8
- removed net CLK-: IC2.DSCLP, R20.1, R21.2, SV3.6
- removed net DAT+: IC2.DSDAP, R16.1, R17.2, SV3.7
- removed net DAT-: IC2.DSDAM, R17.1, R18.2, SV3.5
- removed net N$10: C5.2
- removed net N$13: R13.1
- removed net N$14: R13.2
- removed net N$6: R1.1, R3.1, R5.1, R8.1, R9.2
- removed net N$7: C4.1, R5.2
- removed net N$8: C4.2, R6.2
- removed net N$9: C5.1
- removed net RTD1: R10.2, R2.1
- removed net RTD2: R11.2, R4.1
- removed net RTD3: R12.2, R6.1
- net +5V: now also INPUT.4, R17.2, SJ2.2, SJ4.2, SPARKFUN.VCC; no longer C1.1, C8.1, IC2.EN, IC2.VDD(A), IC2.VDD(B), R10.2, R12.2, R13.2, R19.2, SV3.4
- net GND: now also INPUT.3, LED1.C, PROBE.1, PROBE.5, PROBE.7, SJ1.2, SJ3.2, SPARKFUN.GND; no longer C1.2, C6.2, C7.2, C8.2, IC2.VSS, R18.1, R21.1, R9.1, SV1.1, SV1.5, SV1.7, SV3.3
- net HTR+: now also INPUT.2, PROBE.4, R10.2; no longer SV1.4, SV3.2
- net HTR-: now also INPUT.1, LED2.C, PROBE.3; no longer SV1.3, SV3.1
- net N$1: now also LED1.A, R17.1; no longer C2.1, R1.2
- net N$2: now also LED2.A, R10.1; no longer C2.2, R2.2
- net N$4: now also IC1.ADR1, SJ1.1, SJ2.1; no longer C3.1, R3.2
- net N$5: now also IC1.ADR0, SJ3.1, SJ4.1; no longer C3.2, R4.2
- net RTD0+: now also PROBE.8, R4.1, R6.1; no longer R15.2, R9.1, SV1.8
- net RTD1+: now also PROBE.6; no longer SV1.6
- net RTD2+: now also PROBE.2, R14.2, R9.1; no longer R4.1, R6.1, SV1.2
- net SCL(BYPASS): now also INPUT.6, R16.1, SPARKFUN.SCL; no longer IC2.SCL, R11.1, SV3.10
- net SDA(BYPASS): now also INPUT.5, R11.1, SPARKFUN.SDA; no longer IC2.SDA, R10.1, SV3.9
- net VREF: now also R15.2; no longer R14.2
Other:
- note added: "Indicator LEDs"
- note removed: "Differential 12C Driver"
- moved on the sheet: R10, R11, R16, R17
