File: Sapflow/sapflow_v4/sapflow_v4.brd (EAGLE design)
At the start: 42.5 x 53.3 mm, 47 parts, among them Q1 NMOS, Q4 NMOS, Q5 NMOS, U1 MAXIM_MAX5033BASA+MAXIM_MAX50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

Commit message: Created BOM for orders of 12 boards
Reduced the BOM length by changing some part values on sapflow_v4
Parts:
- R1, R2: value 30k -> 40k
- R11, R12, R13, R14, R3: value 10k -> 5k
- R4: value 100k -> 40k
- R8: value 2k -> 1.5k
- R9: value 820 -> 910
Changed lines of the file:
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@@
 <?xml version="1.0" encoding="utf-8"?>
 <!DOCTYPE eagle SYSTEM "eagle.dtd">
-<eagle version="9.6.0">
+<eagle version="9.5.2">
 <drawing>
 <settings>
@@
 <attribute name="VENDOR" value="Maxim Integrated Products" x="76.542" y="-4.216" size="1.778" layer="27" display="off"/>
 </element>
-<element name="R2" library="rcl" library_urn="urn:adsk.eagle:library:334" package="R0805" package3d_urn="urn:adsk.eagle:package:23553/2" value="30k" x="24.33" y="39.83" smashed="yes" rot="R90">
+<element name="R2" library="rcl" library_urn="urn:adsk.eagle:library:334" package="R0805" package3d_urn="urn:adsk.eagle:package:23553/2" value="40k" x="24.33" y="39.83" smashed="yes" rot="R90">
 <attribute name="NAME" x="24.94" y="37.792" size="0.8128" layer="25" font="vector" ratio="10" rot="R180"/>
 <attribute name="POPULARITY" value="85" x="24.33" y="39.83" size="1.778" layer="27" rot="R90" display="off"/>
 <attribute name="SPICEPREFIX" value="R" x="24.33" y="39.83" size="1.778" layer="27" rot="R90" display="off"/>
 </element>
-<element name="R1" library="rcl" library_urn="urn:adsk.eagle:library:334" package="R0805" package3d_urn="urn:adsk.eagle:package:23553/2" value="30k" x="24.33" y="44.93" smashed="yes" rot="R270">
+<element name="R1" library="rcl" library_urn="urn:adsk.eagle:library:334" package="R0805" package3d_urn="urn:adsk.eagle:package:23553/2" value="40k" x="24.33" y="44.93" smashed="yes" rot="R270">
 <attribute name="NAME" x="23.6246" y="47.1392" size="0.8128" layer="25" font="vector" ratio="10"/>
 <attribute name="POPULARITY" value="85" x="24.33" y="44.93" size="1.778" layer="27" rot="R270" display="off"/>
@@
 <attribute name="NAME" x="27.36" y="39.806" size="0.8128" layer="25" font="vector"/>
 </element>
-<element name="R8" library="rcl" library_urn="urn:adsk.eagle:library:334" package="R0805" package3d_urn="urn:adsk.eagle:package:23553/2" value="2k" x="27.94" y="45.88" smashed="yes">
+<element name="R8" library="rcl" library_urn="urn:adsk.eagle:library:334" package="R0805" package3d_urn="urn:adsk.eagle:package:23553/2" value="1.5k" x="27.94" y="45.88" smashed="yes">
 <attribute name="NAME" x="25.9588" y="47.0738" size="0.8128" layer="25" font="vector" ratio="10"/>
 <attribute name="POPULARITY" value="85" x="27.94" y="45.88" size="1.778" layer="27" display="off"/>
 <attribute name="SPICEPREFIX" value="R" x="27.94" y="45.88" size="1.778" layer="27" display="off"/>
 </element>
-<element name="R9" library="rcl" library_urn="urn:adsk.eagle:library:334" package="R0805" package3d_urn="urn:adsk.eagle:package:23553/2" value="820" x="26.83" y="37.76" smashed="yes" rot="R270">
+<element name="R9" library="rcl" library_urn="urn:adsk.eagle:library:334" package="R0805" package3d_urn="urn:adsk.eagle:package:23553/2" value="910" x="26.83" y="37.76" smashed="yes" rot="R270">
 <attribute name="NAME" x="27.346" y="35.654" size="0.8128" layer="25" font="vector" ratio="10" rot="R180"/>
 <attribute name="POPULARITY" value="85" x="26.83" y="37.76" size="1.778" layer="27" rot="R270" display="off"/>
@@
 <attribute name="VALUE" x="31.435" y="48.398" size="0.0254" layer="27"/>
 </element>
-<element name="R4" library="rcl" library_urn="urn:adsk.eagle:library:334" package="R0805" package3d_urn="urn:adsk.eagle:package:23553/2" value="100k" x="25.23" y="49.53" smashed="yes">
+<element name="R4" library="rcl" library_urn="urn:adsk.eagle:library:334" package="R0805" package3d_urn="urn:adsk.eagle:package:23553/2" value="40k" x="25.23" y="49.53" smashed="yes">
 <attribute name="NAME" x="27.7446" y="49.3014" size="0.8128" layer="25" font="vector" ratio="10"/>
 <attribute name="POPULARITY" value="85" x="25.23" y="49.53" size="1.778" layer="27" display="off"/>
@@
 <attribute name="SPICEPREFIX" value="C" x="11.43" y="63.5" size="1.778" layer="27" rot="R270" display="off"/>
 </element>
-<element name="R3" library="rcl" library_urn="urn:adsk.eagle:library:334" package="R0805" package3d_urn="urn:adsk.eagle:package:23553/2" value="10k" x="3.81" y="40.005" smashed="yes" rot="R90">
+<element name="R3" library="rcl" library_urn="urn:adsk.eagle:library:334" package="R0805" package3d_urn="urn:adsk.eagle:package:23553/2" value="5k" x="3.81" y="40.005" smashed="yes" rot="R90">
 <attribute name="NAME" x="7.0866" y="40.5892" size="1.27" layer="25" font="vector" rot="R180"/>
 <attribute name="POPULARITY" value="85" x="-13.97" y="40.005" size="1.778" layer="27" rot="R90" display="off"/>
@@
 <attribute name="VALUE" x="-4.572" y="7.366" size="0.6096" layer="27" font="vector" ratio="20" rot="R90"/>
 </element>
-<element name="R11" library="rcl" library_urn="urn:adsk.eagle:library:334" package="R0805" package3d_urn="urn:adsk.eagle:package:23553/2" value="10k" x="-6.35" y="20.066" smashed="yes" rot="R270">
+<element name="R11" library="rcl" library_urn="urn:adsk.eagle:library:334" package="R0805" package3d_urn="urn:adsk.eagle:package:23553/2" value="5k" x="-6.35" y="20.066" smashed="yes" rot="R270">
 <attribute name="NAME" x="-5.1308" y="22.0472" size="0.8128" layer="25" font="vector" rot="R270"/>
 <attribute name="POPULARITY" value="85" x="-6.35" y="20.066" size="1.778" layer="27" rot="R270" display="off"/>
 <attribute name="SPICEPREFIX" value="R" x="-6.35" y="20.066" size="1.778" layer="27" rot="R270" display="off"/>
 </element>
-<element name="R12" library="rcl" library_urn="urn:adsk.eagle:library:334" package="R0805" package3d_urn="urn:adsk.eagle:package:23553/2" value="10k" x="5.08" y="10.16" smashed="yes">
+<element name="R12" library="rcl" library_urn="urn:adsk.eagle:library:334" package="R0805" package3d_urn="urn:adsk.eagle:package:23553/2" value="5k" x="5.08" y="10.16" smashed="yes">
 <attribute name="NAME" x="3.8608" y="11.2268" size="0.8128" layer="25" font="vector"/>
 <attribute name="POPULARITY" value="85" x="5.08" y="10.16" size="1.778" layer="27" display="off"/>
 <attribute name="SPICEPREFIX" value="R" x="5.08" y="10.16" size="1.778" layer="27" display="off"/>
 </element>
-<element name="R13" library="rcl" library_urn="urn:adsk.eagle:library:334" package="R0805" package3d_urn="urn:adsk.eagle:package:23553/2" value="10k" x="7.366" y="5.588" smashed="yes" rot="R90">
+<element name="R13" library="rcl" library_urn="urn:adsk.eagle:library:334" package="R0805" package3d_urn="urn:adsk.eagle:package:23553/2" value="5k" x="7.366" y="5.588" smashed="yes" rot="R90">
 <attribute name="NAME" x="8.5598" y="8.6868" size="0.8128" layer="25" font="vector" rot="R180"/>
 <attribute name="POPULARITY" value="85" x="7.366" y="5.588" size="1.778" layer="27" rot="R90" display="off"/>
 <attribute name="SPICEPREFIX" value="R" x="7.366" y="5.588" size="1.778" layer="27" rot="R90" display="off"/>
 </element>
-<element name="R14" library="rcl" library_urn="urn:adsk.eagle:library:334" package="R0805" package3d_urn="urn:adsk.eagle:package:23553/2" value="10k" x="1.016" y="10.16" smashed="yes" rot="R180">
+<element name="R14" library="rcl" library_urn="urn:adsk.eagle:library:334" package="R0805" package3d_urn="urn:adsk.eagle:package:23553/2" value="5k" x="1.016" y="10.16" smashed="yes" rot="R180">
 <attribute name="NAME" x="2.0066" y="12.065" size="0.8128" layer="25" font="vector" rot="R180"/>
 <attribute name="POPULARITY" value="85" x="1.016" y="10.16" size="1.778" layer="27" rot="R180" display="off"/>
