File: Sapflow/sapflow_v4/sapflow_v4.sch (EAGLE design)
At the start: 47 parts, among them Q1 NMOS, Q4 NMOS, Q5 NMOS, U1 MAXIM_MAX5033BASA+MAXIM_MAX50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

Commit message: Created BOM for orders of 12 boards
Reduced the BOM length by changing some part values on sapflow_v4
Parts:
- R1, R2: value 30k -> 40k
- R11, R12, R13, R14, R3: value 10k -> 5k
- R4: value 100k -> 40k
- R8: value 2k -> 1.5k
- R9: value 820 -> 910
