File: Sapflow/sapflow_v5/sapflow_v5.sch (EAGLE design)
At the start: 47 parts, among them Q1 NMOS, Q4 NMOS, Q5 NMOS, U1 MAXIM_MAX5033BASA+MAXIM_MAX50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

Commit message: changed to v5 of sapflow wing
Parts:
- removed 3V|5V: (no value), SparkFun-Connectors:CONN_021X02_NO_SILK
- removed JP1: (no value), adafruit:PINHD-1X1CB
- removed LED2: RED, adafruit:LEDCHIPLED_0805
- removed MS1: FEATHERWING, powerboard:FEATHERWING
- removed R9: 910, rcl:R-US_R0805
- removed TP1, TP2: TPTP16R, testpad:TPTP16R
- added LED3: RED, adafruit:LEDCHIPLED_0805
- added R5: 910, rcl:R-US_R0805
- added R6: 40k, rcl:R-US_R0805
- MICROSD: device adafruit:MICROSD -> adafruit_improved:MICROSD
Connections:
- net +12V renamed 12V
- net +3V3 renamed 3V3
- net 5VUSB renamed 5V
- net N$1 renamed 5V_EN
- net N$3 renamed 3V_EN
- removed net A3: MS1.GPIOA3, MS2.GPIOA3, T2.G
- removed net N$13: LED2.A, R9.1
- removed net N$7: MS1.GPIO6
- removed net N$8: MS1.GPIO5
- removed net RESET: MS1.!RESET, MS2.!RESET, U$1.P$2
- new net HTR_EN: MS2.GPIOA3, R6.2, T2.G
- new net N$1: MS2.!RESET, U$1.P$2
- new net N$5: LED3.A, R5.1
- net 0RX: no longer MS1.GPIORX
- net 11: no longer MS1.GPIO11
- net 13: no longer MS1.GPIO13
- net 1TX: no longer MS1.GPIOTX
- net 3VRAIL: now also R5.2; no longer 3V|5V.1, MS1.3V, R9.2
- net 5VRAIL: no longer 3V|5V.2, MS1.USB
- net 9: no longer MS1.GPIO9
- net A0: no longer MS1.GPIOA0
- net A1: no longer MS1.GPIOA1
- net A2: no longer MS1.GPIOA2
- net A4: no longer MS1.GPIOA4
- net A5: no longer MS1.GPIOA5
- net ARF: no longer MS1.AREF
- net CLK: no longer MS1.GPIOSCK
- net DFU: no longer MS1.NC
- net DI: no longer MS1.GPIOMOSI
- net DO: no longer MS1.GPIOMISO
- net EN: no longer MS1.EN, TP1.TP
- net GND: now also LED3.C, R6.1; no longer JP1.1, LED2.C, MS1.GND, TP2.TP
- net N$11: no longer MS1.GPIO10
- net N$14: no longer MS1.GPIO12
- net SCL: no longer MS1.GPIOSCL
- net SCL_5: now also PROBE.5; no longer PROBE.3
- net SDA: no longer MS1.GPIOSDA
- net SDA_5: now also PROBE.3; no longer PROBE.5
- net VBATT: no longer MS1.VBAT
Other:
- note added: "Manual RTC Wake Up"
- note removed: "Change from V1 to V2: RTC is powered with 3v3 instead of Vbat Add red LED if rail are switched on"
- note removed: "Decoupling"
- note removed: "Handle Max 0.4 A"
- note removed: "Manually Wake Up (Testing purpose_)"
- note removed: "Manually probing headers (testing purpose)"
- moved on the sheet: B1, BATTERY, C1, C2, C3, C5, C6, C7, C8, CS, D1, D2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
